File: breadebyte.kicad/breadebyte.kicad_sch (KiCad schematic)
At the start: 6 parts, among them J1 USB_B_Micro, J2 Conn_Left, J3 Conn_Right, J4 SWD, U1 E73-2G4M08S1E

Commit message: Switch to using shared symbol/footprint library
Parts:
- J1: footprint breadebyte:USB_Micro-B_HRO_U-D-M5DD-W-1_Vertical -> spbnick:USB_Micro-B_HRO_U-D-M5DD-W-1_Vertical
- U1: footprint breadebyte:E73-2G4M08S1E -> spbnick:E73-2G4M08S1E; symbol breadebyte:E73-2G4M08S1E -> spbnick:E73-2G4M08S1E
Changed lines of the file:
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@@
     (effects (font (size 1.27 1.27)) (justify right bottom))
   )
-  (symbol (lib_id "breadebyte:E73-2G4M08S1E") (at 63.5 90.17 0) (unit 1)
+  (symbol (lib_id "spbnick:E73-2G4M08S1E") (at 63.5 90.17 0) (unit 1)
     (in_bom yes) (on_board yes)
     (property "Reference" "U1" (id 0) (at 52.07 59.69 0))
     (property "Value" "E73-2G4M08S1E" (id 1) (at 76.2 59.69 0))
-    (property "Footprint" "breadebyte:E73-2G4M08S1E" (id 2) (at 82.55 118.11 0)
-      (effects (font (size 1.27 1.27)) hide)
-    )
-    (property "Datasheet" "https://www.espressif.com/sites/default/files/documentation/esp32-s2-wroom_esp32-s2-wroom-i_datasheet_en.pdf" (id 3) (at 55.88 110.49 0)
+    (property "Footprint" "spbnick:E73-2G4M08S1E" (id 2) (at 82.55 118.11 0)
+      (effects (font (size 1.27 1.27)) hide)
+    )
+    (property "Datasheet" "https://www.ebyte.com/en/downpdf.aspx?id=1035" (id 3) (at 55.88 110.49 0)
       (effects (font (size 1.27 1.27)) hide)
     )
@@
     (property "Reference" "J1" (id 0) (at 166.5478 21.1582 0))
     (property "Value" "USB_B_Micro" (id 1) (at 166.5478 23.4696 0))
-    (property "Footprint" "breadebyte:USB_Micro-B_HRO_U-D-M5DD-W-1_Vertical" (id 2) (at 168.91 34.29 0)
+    (property "Footprint" "spbnick:USB_Micro-B_HRO_U-D-M5DD-W-1_Vertical" (id 2) (at 168.91 34.29 0)
       (effects (font (size 1.27 1.27)) hide)
     )
@@
     )
     (path "/00000000-0000-0000-0000-000061b36174"
-      (reference "J1") (unit 1) (value "USB_B_Micro") (footprint "breadebyte:USB_Micro-B_HRO_U-D-M5DD-W-1_Vertical")
+      (reference "J1") (unit 1) (value "USB_B_Micro") (footprint "spbnick:USB_Micro-B_HRO_U-D-M5DD-W-1_Vertical")
     )
     (path "/00000000-0000-0000-0000-000061b70745"
@@
     )
     (path "/00000000-0000-0000-0000-000061aec9bf"
-      (reference "U1") (unit 1) (value "E73-2G4M08S1E") (footprint "breadebyte:E73-2G4M08S1E")
-    )
-  )
+      (reference "U1") (unit 1) (value "E73-2G4M08S1E") (footprint "spbnick:E73-2G4M08S1E")
+    )
+  )
